Commit message: Kinect libaries added

File: ros/src/robot_model/urdf/robot_model.xacro (robot description, xacro)
@@ -1,156 +1,13 @@
 <?xml version='1.0'?>
 <robot name="robot_model" xmlns:xacro="http://www.ros.org/wiki/xacro">
-  <xacro:include filename="$(find robot_model)/urdf/robot_model.gazebo" />
-  <link name="robot_footprint"></link>
-  <joint name="robot_footprint_joint" type="fixed">
-    <origin xyz="0 0 0" rpy="0 0 0" />
-    <parent link="robot_footprint"/>
-    <child link="chassis" />
-  </joint>
-  <link name='chassis'>
-    <pose>0 0 0.1 0 0 0</pose>
-    <inertial>
-      <mass value="15.0"/>
-      <origin xyz="-0.2 0 0" rpy=" 0 0 0"/>
-      <inertia
-          ixx="0.1" ixy="0" ixz="0"
-          iyy="0.1" iyz="0"
-          izz="0.1"
-      />
-    </inertial>
-    <collision name='collision'>
-      <origin xyz="0.1 0 0" rpy=" 0 0 0"/>
-      <geometry>
-        <box size="1.2 .64 .07"/>
-      </geometry>
-    </collision>
-    <visual name='chassis_visual'>
-      <origin xyz="0.1 0 0" rpy=" 0 0 0"/>
-      <geometry>
-        <box size="1.2 .64 .07"/>
-      </geometry>
-    </visual>
-    <collision name='front_caster_collision'>
-      <origin xyz="0.45 0 -0.035" rpy=" 0 0 0"/>
-      <geometry>
-        <sphere radius="0.0499"/>
-      </geometry>
-    <surface>
-    <friction>
-    <ode>
-        <mu>0</mu>
-        <mu2>0</mu2>
-        <slip1>1.0</slip1>
-        <slip2>1.0</slip2>
-    </ode>
-    </friction>
-    </surface>
-    </collision>
-    <visual name='front_caster_visual'>
-      <origin xyz="0.45 0 -0.035" rpy=" 0 0 0"/>
-      <geometry>
-        <sphere radius="0.05"/>
-      </geometry>
-    </visual>
+  <link name='base_link'>
   </link>
-  <link name='left_wheel'>
-    <inertial>
-          <mass value="5.0"/>
-          <origin xyz="0.0 0 0" rpy=" 0 1.5705 1.5705"/>
-          <inertia
-              ixx="0.1" ixy="0" ixz="0"
-              iyy="0.1" iyz="0"
-              izz="0.1"
-          />
-    </inertial>
-    <collision name='left_wheel_collision'>
-      <origin xyz="0 0 0" rpy=" 0 1.5707 1.5707"/>
-      <geometry>
-          <cylinder radius="0.085" length="0.1"/>
-      </geometry>
-    </collision>
-    <visual name='left_wheel_visual'>
-      <origin xyz="0 0 0" rpy=" 0 1.5707 1.5707"/>
-      <geometry>
-          <cylinder radius="0.085" length="0.1"/>
-      </geometry>
-    </visual>
+  <link name='camera_link'>
   </link>
-  <link name='right_wheel'>
-    <inertial>
-          <mass value="5.0"/>
-          <origin xyz="0.0 0 0" rpy=" 0 1.5705 1.5705"/>
-          <inertia
-              ixx="0.1" ixy="0" ixz="0"
-              iyy="0.1" iyz="0"
-              izz="0.1"
-          />
-    </inertial>
-    <collision name='collision'>
-      <origin xyz="0 0 0" rpy=" 0 1.5707 1.5707"/>
-      <geometry>
-          <cylinder radius="0.085" length="0.1"/>
-      </geometry>
-    </collision>
-    <visual name='visual'>
-      <origin xyz="0 0 0" rpy=" 0 1.5707 1.5707"/>
-      <geometry>
-          <cylinder radius="0.085" length="0.1"/>
-      </geometry>
-    </visual>
-  </link>
-  <link name='kinect'>
-      <inertial>
-        <mass value="1e-5"/>
-        <origin xyz="0.0 0 0" rpy=" 0 0 0"/>
-        <inertia
-            ixx="1e-6" ixy="0" ixz="0"
-            iyy="1e-6" iyz="0"
-            izz="1e-6"
-        />
-      </inertial>
-      <collision name='collision'>
-        <origin xyz="0 0 0" rpy=" 0 0 0"/>
-        <geometry>
-            <box size="0.1 0.1 0.1"/>
-        </geometry>
-      </collision>
-      <visual name='visual'>
-        <origin xyz="0 0 0" rpy=" 0 0 0"/>
-        <geometry>
-            <mesh filename="package://robot_model/meshes/hokuyo.dae"/>
-        </geometry>
-      </visual>
-  </link>
-  <joint type="continuous" name="left_wheel_hinge">
-    <origin xyz="-0.490 0.375 0.0" rpy="0 0 0"/>
-    <child link="left_wheel"/>
-    <parent link="chassis"/>
-    <axis xyz="0 1 0" rpy="0 0 0"/>
-    <limit effort="100" velocity="100"/>
-    <dynamics damping="1.0" friction="1.0"/>
-  </joint>
-  <joint type="continuous" name="right_wheel_hinge">
-      <origin xyz="-0.490 -0.375 0.0" rpy="0 0 0"/>
-      <child link="right_wheel"/>
-      <parent link="chassis"/>
-      <axis xyz="0 1 0" rpy="0 0 0"/>
-      <limit effort="100" velocity="1000"/>
-      <dynamics damping="1.0" friction="1.0"/>
-  </joint>
   <joint type="fixed" name="kinect_joint">
     <origin xyz="0.25 0 0.02" rpy="0 0 0"/>
-    <child link="hokuyo"/>
-    <parent link="chassis"/>
+    <child link="camera_link"/>
+    <parent link="base_link"/>
     <axis xyz="0 1 0" rpy="0 0 0"/>
   </joint>
-  <gazebo reference="left_wheel">
-      <material>Gazebo/Green</material>
-  </gazebo>
-  <gazebo reference="right_wheel">
-      <material>Gazebo/Green</material>
-  </gazebo>
-  <gazebo reference="camera">
-      <material>Gazebo/Red</material>
-  </gazebo>
 </robot>
